File: ts_23_LV_BMS_MASTER/LV_MASTER_A_SAMPLE/MCU.kicad_sch (KiCad schematic)
At the start: 27 parts, among them J2 UART, J3 BOOT1, J4 STLINK, U1 STM32F446RET7, Y1 ECS-80-18-30-JGN-TR, Y2 FC-135_32.7680KA-A5

Commit message: Minor Changes
Parts:
- gave numbers to parts that had none: 1
Changed lines of the file:
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@@
   (symbol (lib_id "ERJP06F1000V:ERJP06F1000V") (at 135.89 175.26 270) (unit 1)
     (in_bom yes) (on_board yes)
-    (property "Reference" "R?" (id 0) (at 139.7 186.69 90))
+    (property "Reference" "R29" (id 0) (at 139.7 186.69 90))
     (property "Value" "50mR" (id 1) (at 139.7 184.15 90))
     (property "Footprint" "Resistor_SMD:R_0603_1608Metric_Pad0.98x0.95mm_HandSolder" (id 2) (at 137.16 189.23 0)
