File: ts_23_LV_BMS_MASTER/LV_MASTER_A_SAMPLE/LV_MASTER_A_SAMPLE.kicad_pcb (KiCad board)
At the start: 4 copper layers, 77.5 x 46.9 mm, 117 parts, among them J1 DT 12P, J2 UART, J3 BOOT1, J4 STLINK, J5 Conn_01x02_Male, J6 Conn_02x02_Counter_Clockwise, J7 Conn_02x02_Counter_Clockwise, Q1 STD7NK40Z, Q2 STD7NK40Z, T1 HX1188NL, U1 STM32F446RET7, U2 TLV70033_SOT23-5, U4 ADM3053, U5 B82786C0104H002, U6 LTC6820, U7 ISO1540, U8 ADS1115, U9 ADUM3221, Y1 ECS-80-18-30-JGN-TR, Y2 FC-135_32.7680KA-A5

Commit message: Last Minute Changes
Parts:
- added U3: R-78C5.0-1.0, Converter_DCDC:Converter_DCDC_RECOM_R-78E-0.5_THT, B.Cu at (168.8, 91.5)
- TP1: renamed from AUX_OUT; value AUX_OUT -> TestPoint
- TP2: renamed from BL_RLY; value BL_RLY -> TestPoint
- moved C49 1.36 mm to (165.8, 94.5)
- moved J1 0.15 mm to (177.3, 91.0)
Routing:
- net +24V: track 51.3 -> 55.9 mm, vias 1 -> 0
- net +5V: track 36.4 -> 40.3 mm, vias 6 -> 5
- net /GLV+: track 17.0 -> 16.0 mm
- net GND: vias 212 -> 209

Commit message: Final Changes to board
Parts:
- removed D10, D9: LED, LED_SMD:LED_0805_2012Metric_Pad1.15x1.40mm_HandSolder
- removed D7, D8: SD560BTR, Diode_SMD:D_SMB_Handsoldering
- removed Q1, Q2: STD7NK40Z, Package_TO_SOT_SMD:TO-252-2
- removed R24, R26: 20.0K, Resistor_SMD:R_0603_1608Metric_Pad0.98x0.95mm_HandSolder
- removed R25, R27: 1.5k, Resistor_SMD:R_0603_1608Metric_Pad0.98x0.95mm_HandSolder
- removed TP1, TP2: TestPoint, TestPoint:TestPoint_Pad_1.0x1.0mm
- added 11: IXDN604SIA, BMS_Library:SOIC127P600X175-8N, F.Cu at (163.6, 103.8)
- added C54: 10uF, Capacitor_SMD:C_0603_1608Metric_Pad1.08x0.95mm_HandSolder, F.Cu at (169.2, 105.7)
- added C55: 10.0nF, Capacitor_SMD:C_0603_1608Metric_Pad1.08x0.95mm_HandSolder, F.Cu at (165.1, 108.4)
- added C56: 10.0nF, Capacitor_SMD:C_0603_1608Metric_Pad1.08x0.95mm_HandSolder, F.Cu at (162.3, 107.5)
- added L2: 12uH, Inductor_SMD:L_1210_3225Metric_Pad1.42x2.65mm_HandSolder, F.Cu at (153.8, 92.6)
- C20: footprint Capacitor_SMD:C_0805_2012Metric_Pad1.18x1.45mm_HandSolder -> BMS_Library:TLV_10X10.5_; moved to F.Cu
- C53: value 10.0uF -> 0.1uF
- J1: moved to B.Cu
- U9: value ADUM3221 -> ADuM120N
- moved C53 23.3 mm to (171.5, 105.7), turned to 90 degrees
- moved U3 17.9 mm to (152.9, 99.8), turned to 0 degrees
- moved C20 17.3 mm to (164.5, 92.5)
- moved C49 8.99 mm to (156.8, 95.1)
- moved C35 3.39 mm to (166.9, 83.1), turned to 180 degrees
- moved C34 2.95 mm to (163.2, 83.7)
- moved C31 2.90 mm to (156.8, 86.4)
- moved C32 2.90 mm to (155.1, 86.4)
- moved C29 2.90 mm to (156.6, 75.8)
- moved C30 2.90 mm to (154.9, 75.8)
- moved C33 2.90 mm to (163.2, 77.2)
- moved R5 2.90 mm to (158.5, 75.8)
- moved U5 2.90 mm to (164.1, 80.0)
- moved D6 2.90 mm to (158.0, 80.5)
- moved U4 2.90 mm to (147.1, 81.1)
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Connections:
- net /CAN1_H renamed /CAN1 +
- net /CAN1_L renamed /CAN1 -
- C22 pad 1: +24V -> Net-(L1-Pad2)
- C51 pad 2: 5V_(ISO) -> +3.3V
- C53 pad 2: +5V -> +24V
- J7 pad 1: /BLUE_LOOP_RLY -> /AUX_OUTPUT
- J7 pad 2: /AUX_OUTPUT -> /BLUE_LOOP_RLY
- L1 pad 2: +24V -> Net-(L1-Pad2)
- U9 pad 1: 5V_(ISO) -> +3.3V
- U9 pad 6: /Blue Loop/VOB -> /Blue Loop/IN2
- U9 pad 7: /Blue Loop/VOA -> /Blue Loop/IN1
Routing:
- net +24V: track 55.9 -> 31.8 mm, vias 0 -> 1
- net /GLV+: track 16.0 -> 36.0 mm
- net /Blue Loop/IN2: track 0.00 -> 18.6 mm
- net /Blue Loop/IN1: track 0.00 -> 17.1 mm
- net /Blue Loop/VOA: track 12.9 -> 0.00 mm
- net /Blue Loop/VOB: track 12.4 -> 0.00 mm, vias 1 -> 0
- net /AUX_OUTPUT: track 20.1 -> 8.38 mm
- net /CAN1 +: track 16.0 -> 4.88 mm
- net +5V: track 40.3 -> 29.3 mm
- net Net-(C20-Pad1): track 9.77 -> 20.3 mm, vias 0 -> 1
- net Net-(L1-Pad2): track 0.00 -> 8.40 mm, vias 0 -> 1
- net +3.3V: track 0.00 -> 2.87 mm, vias 0 -> 1
- net /CAN1 -: track 7.41 -> 5.30 mm
- net Net-(D10-Pad2): track 2.00 -> 0.00 mm
- net Net-(D9-Pad2): track 1.97 -> 0.00 mm
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