File: ts_23_LV_BMS_MASTER/LV_MASTER_A_SAMPLE/LV_MASTER_A_SAMPLE.kicad_sch (KiCad schematic)
At the start: 4 parts, among them J1 DT 12P, J5 Conn_01x02_Male, J6 Conn_02x02_Counter_Clockwise, J7 Conn_02x02_Counter_Clockwise

Commit message: Final Changes to board
Connections:
- net AUX_OUTPUT: now also J7.1 (Pin_1); no longer J7.2 (Pin_2)
- net BLUE_LOOP_RLY: now also J7.2 (Pin_2); no longer J7.1 (Pin_1)
- net CAN1_H renamed CAN1 +
- net CAN1_L renamed CAN1 -
