File: ts_23_LV_BMS_MASTER/LV_MASTER_A_SAMPLE/Power.kicad_sch (KiCad schematic)
At the start: 21 parts, among them U2 TLV70033_SOT23-5, U3 R-78C5.0-1.0

Commit message: Final Changes to board
Parts:
- added L2: 12uH, Inductor_SMD:L_1210_3225Metric_Pad1.42x2.65mm_HandSolder, symbol Device:L_Small
- C20: footprint Capacitor_SMD:C_0805_2012Metric_Pad1.18x1.45mm_HandSolder -> BMS_Library:TLV_10X10.5_
Connections:
- net +24V: now also L2.2; no longer C22.1, L1.2 (4)
- new net: C22.1, L1.2 (4), L2.1
Other:
- moved on the sheet: C22, C23
